File: Motor Driver.kicad_sch (KiCad schematic)
At the start: 9 parts, among them J1 Conn_01x02, U2 DRV8801PWP

Commit message: Add 10k pulldown to nSleep and export BOM
Parts:
- C3: Mfr. No (none) -> UVZ1J101MPD
Changed lines of the file:
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@@
+      (effects (font (size 1.27 1.27)) hide)
+    )
+    (property "Mfr. No" "UVZ1J101MPD" (at 31.75 30.48 90)
       (effects (font (size 1.27 1.27)) hide)
     )

Commit message: Update 0.1uF capacitor mfr no
Parts:
- C1, C2, C4: Mfr. No KGM21NR71E104KT -> 08055C104JAT2A
Changed lines of the file:
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@@
       (effects (font (size 1.27 1.27)) hide)
     )
-    (property "Mfr. No" "KGM21NR71E104KT" (at 31.75 38.1 90)
+    (property "Mfr. No" "08055C104JAT2A" (at 31.75 38.1 90)
       (effects (font (size 1.27 1.27)) hide)
     )
@@
       (effects (font (size 1.27 1.27)) hide)
     )
-    (property "Mfr. No" "KGM21NR71E104KT" (at 35.56 46.99 0)
+    (property "Mfr. No" "08055C104JAT2A" (at 35.56 46.99 0)
       (effects (font (size 1.27 1.27)) hide)
     )
@@
       (effects (font (size 1.27 1.27)) hide)
     )
-    (property "Mfr. No" "KGM21NR71E104KT" (at 43.18 40.64 90)
-      (effects (font (size 1.27 1.27)) hide)
-    )
+    (property "Mfr. No" "08055C104JAT2A" (at 43.18 40.64 90)
+      (effects (font (size 1.27 1.27)) hide)
+    )

Commit message: Change Screw Terminal Part and update Mfr No's
Parts:
- J1: footprint TerminalBlock_Phoenix:TerminalBlock_Phoenix_MKDS-1,5-2-5.08_1x02_P5.08mm_Horizontal -> TB009-508-02BE:CUI_TB009-508-02BE; Mfr. No (none) -> TB009-508-02BE
- U2: Mfr. No (none) -> DRV8801PWP
Changed lines of the file:
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@@
       (effects (font (size 1.27 1.27)) (justify left))
     )
-    (property "Footprint" "TerminalBlock_Phoenix:TerminalBlock_Phoenix_MKDS-1,5-2-5.08_1x02_P5.08mm_Horizontal" (at 105.41 38.1 0)
+    (property "Footprint" "TB009-508-02BE:CUI_TB009-508-02BE" (at 105.41 38.1 0)
       (effects (font (size 1.27 1.27)) hide)
     )
     (property "Datasheet" "~" (at 105.41 38.1 0)
+      (effects (font (size 1.27 1.27)) hide)
+    )
+    (property "Mfr. No" "TB009-508-02BE" (at 105.41 38.1 0)
       (effects (font (size 1.27 1.27)) hide)
     )
@@
       (effects (font (size 1.27 1.27)) hide)
     )
+    (property "Mfr. No" "DRV8801PWP" (at 68.58 48.26 0)
+      (effects (font (size 1.27 1.27)) hide)
+    )

Commit message: Add mouser no's, pullup resistor, change project name
Parts:
- C1, C2, C4: Mouser No (none) -> 581-08055C104J
- C19: Mouser No (none) -> 581-KAF21BR72D102MT
- C3: Mouser No (none) -> 647-UVZ1J101MPD
- J1: Mouser No (none) -> 490-TB009-508-02BE
- R1: Mouser No (none) -> 667-ERJ-D1CFR200U
- R5: Mouser No (none) -> 652-CRS0805FX1002ELF
- U2: value DRV8801PWP -> DRV8801PWPR; Mfr. No DRV8801PWP -> DRV8801PWPR; Mouser No (none) -> 595-DRV8801PWPR
Changed lines of the file:
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@@
       (effects (font (size 1.27 1.27)) hide)
     )
-    (pin "1")
-    (pin "2")
-    (instances
-      (project "BioRobotics Tank PCB"
+    (property "Mouser No" "581-08055C104J" (at 31.75 38.1 0)
+      (effects (font (size 1.27 1.27)) hide)
+    )
+    (pin "1")
+    (pin "2")
+    (instances
+      (project "PicoDrive"
         (path "/738c766b-5149-4d22-8944-003aead1c6f2/91fbf09a-497d-4de7-ab4a-2985c5e3b4aa"
           (reference "C1") (unit 1)
@@
       (effects (font (size 1.27 1.27)) hide)
     )
-    (pin "1")
-    (pin "2")
-    (instances
-      (project "BioRobotics Tank PCB"
+    (property "Mouser No" "581-KAF21BR72D102MT" (at 99.06 62.23 0)
+      (effects (font (size 1.27 1.27)) hide)
+    )
+    (pin "1")
+    (pin "2")
+    (instances
+      (project "PicoDrive"
         (path "/738c766b-5149-4d22-8944-003aead1c6f2/91fbf09a-497d-4de7-ab4a-2985c5e3b4aa"
           (reference "C19") (unit 1)
@@
       (effects (font (size 1.27 1.27)) hide)
     )
-    (pin "1")
-    (pin "2")
-    (instances
-      (project "BioRobotics Tank PCB"
+    (property "Mouser No" "581-08055C104J" (at 35.56 46.99 0)
+      (effects (font (size 1.27 1.27)) hide)
+    )
+    (pin "1")
+    (pin "2")
+    (instances
+      (project "PicoDrive"
         (path "/738c766b-5149-4d22-8944-003aead1c6f2/91fbf09a-497d-4de7-ab4a-2985c5e3b4aa"
           (reference "C4") (unit 1)
@@
       (effects (font (size 1.27 1.27)) hide)
     )
-    (pin "1")
-    (pin "2")
-    (instances
-      (project "BioRobotics Tank PCB"
+    (property "Mouser No" "652-CRS0805FX1002ELF" (at 91.44 55.88 0)
+      (effects (font (size 1.27 1.27)) hide)
+    )
+    (pin "1")
+    (pin "2")
+    (instances
+      (project "PicoDrive"
         (path "/738c766b-5149-4d22-8944-003aead1c6f2"
           (reference "R5") (unit 1)
@@
     (pin "1")
     (instances
-      (project "BioRobotics Tank PCB"
+      (project "PicoDrive"
         (path "/738c766b-5149-4d22-8944-003aead1c6f2/91fbf09a-497d-4de7-ab4a-2985c5e3b4aa"
           (reference "#PWR024") (unit 1)
@@
       (effects (font (size 1.27 1.27)) hide)
     )
-    (pin "1")
-    (pin "2")
-    (instances
-      (project "BioRobotics Tank PCB"
+    (property "Mouser No" "490-TB009-508-02BE" (at 105.41 38.1 0)
+      (effects (font (size 1.27 1.27)) hide)
+    )
+    (pin "1")
+    (pin "2")
+    (instances
+      (project "PicoDrive"
         (path "/738c766b-5149-4d22-8944-003aead1c6f2/91fbf09a-497d-4de7-ab4a-2985c5e3b4aa"
           (reference "J1") (unit 1)
@@
       (effects (font (size 1.27 1.27)) hide)
     )
-    (pin "1")
-    (pin "2")
-    (instances
-      (project "BioRobotics Tank PCB"
+    (property "Mouser No" "581-08055C104J" (at 43.18 40.64 0)
+      (effects (font (size 1.27 1.27)) hide)
+    )
+    (pin "1")
+    (pin "2")
+    (instances
+      (project "PicoDrive"
         (path "/738c766b-5149-4d22-8944-003aead1c6f2/91fbf09a-497d-4de7-ab4a-2985c5e3b4aa"
           (reference "C2") (unit 1)
@@
       (effects (font (size 1.27 1.27)) hide)
     )
-    (pin "1")
-    (pin "2")
-    (instances
-      (project "BioRobotics Tank PCB"
+    (property "Mouser No" "647-UVZ1J101MPD" (at 31.75 30.48 0)
+      (effects (font (size 1.27 1.27)) hide)
+    )
+    (pin "1")
+    (pin "2")
+    (instances
+      (project "PicoDrive"
         (path "/738c766b-5149-4d22-8944-003aead1c6f2/91fbf09a-497d-4de7-ab4a-2985c5e3b4aa"
           (reference "C3") (unit 1)
@@
     (pin "1")
     (instances
-      (project "BioRobotics Tank PCB"
+      (project "PicoDrive"
         (path "/738c766b-5149-4d22-8944-003aead1c6f2/91fbf09a-497d-4de7-ab4a-2985c5e3b4aa"
           (reference "#PWR03") (unit 1)
@@
       (effects (font (size 1.27 1.27)) hide)
     )
-    (pin "1")
-    (pin "2")
-    (instances
-      (project "BioRobotics Tank PCB"
+    (property "Mouser No" "667-ERJ-D1CFR200U" (at 101.6 45.72 0)
+      (effects (font (size 1.27 1.27)) hide)
+    )
+    (pin "1")
+    (pin "2")
+    (instances
+      (project "PicoDrive"
         (path "/738c766b-5149-4d22-8944-003aead1c6f2/91fbf09a-497d-4de7-ab4a-2985c5e3b4aa"
           (reference "R1") (unit 1)
@@
     (pin "1")
     (instances
-      (project "BioRobotics Tank PCB"
+      (project "PicoDrive"
         (path "/738c766b-5149-4d22-8944-003aead1c6f2/91fbf09a-497d-4de7-ab4a-2985c5e3b4aa"
           (reference "#PWR04") (unit 1)
@@
     (pin "1")
     (instances
-      (project "BioRobotics Tank PCB"
+      (project "PicoDrive"
         (path "/738c766b-5149-4d22-8944-003aead1c6f2/91fbf09a-497d-4de7-ab4a-2985c5e3b4aa"
           (reference "#PWR01") (unit 1)
@@
       (effects (font (size 1.27 1.27)))
     )
-    (property "Value" "DRV8801PWP" (at 68.58 34.29 0)
+    (property "Value" "DRV8801PWPR" (at 68.58 34.29 0)
       (effects (font (size 1.27 1.27)))
     )
@@
       (effects (font (size 1.27 1.27)) hide)
     )
-    (property "Mfr. No" "DRV8801PWP" (at 68.58 48.26 0)
+    (property "Mfr. No" "DRV8801PWPR" (at 68.58 48.26 0)
+      (effects (font (size 1.27 1.27)) hide)
+    )
+    (property "Mouser No" "595-DRV8801PWPR" (at 68.58 48.26 0)
       (effects (font (size 1.27 1.27)) hide)
     )
@@
     (pin "9")
     (instances
-      (project "BioRobotics Tank PCB"
+      (project "PicoDrive"
         (path "/738c766b-5149-4d22-8944-003aead1c6f2/91fbf09a-497d-4de7-ab4a-2985c5e3b4aa"
           (reference "U2") (unit 1)
@@
     (pin "1")
     (instances
-      (project "BioRobotics Tank PCB"
+      (project "PicoDrive"
         (path "/738c766b-5149-4d22-8944-003aead1c6f2/91fbf09a-497d-4de7-ab4a-2985c5e3b4aa"
           (reference "#PWR02") (unit 1)
